File: hw/timelapse.sch (KiCad schematic (older format))
At the start: 37 parts, among them P101 CONN_01X03, Q102 Raltron_32_768kHz_R26, Q103 IRLML6402, SW101 SWITCH_DT, SW102 SW_PUSH, SW103 SW_PUSH, SW104 SW_PUSH, SW105 SW_PUSH, U101 MSP430G2553, U102 Cosmo_1010-817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

Commit message: Add external trigger capability (remove LCD CS line)
Parts:
- added D? (x2): SD103A, symbol SD103A
- added P?: CONN_01X02, symbol CONN_01X02
- CONN101: symbol USB_MINI_B_GMe -> USB_MINI_B_GMe-RESCUE-timelapse
Connections:
- net labels added: ~EXT_TRIGGER
- net labels removed: ~LCD_CS
- wire segments 110 -> 113
Changed lines of the file:
@@
 Text Label 7650 5850 0    60   ~ 0
 D~C
-Text Label 7650 5950 0    60   ~ 0
-~LCD_CS
 $Comp
 L IRLML6402 Q103
@@
 Wire Wire Line
 	5450 6050 5900 6050
-Text Label 5600 5950 0    60   ~ 0
-~LCD_CS
 Wire Wire Line
 	5450 6250 5900 6250
@@
 	800  4200 800  4250
 $Comp
-L USB_MINI_B_GMe CONN101
+L USB_MINI_B_GMe-RESCUE-timelapse CONN101
 U 1 1 57668B1C
 P 1100 2900
@@
 Wire Wire Line
 	2450 6000 2450 5950
+$Comp
+L GND #PWR?
+U 1 1 579CBEAE
+P 7650 5950
+F 0 "#PWR?" H 7650 5700 50  0001 C CNN
+F 1 "GND" H 7650 5800 50  0000 C CNN
+F 2 "" H 7650 5950 60  0000 C CNN
+F 3 "" H 7650 5950 60  0000 C CNN
+	1    7650 5950
+	1    0    0    -1
+$EndComp
+Text Label 5600 5950 0    60   ~ 0
+~EXT_TRIGGER
+$Comp
+L CONN_01X02 P?
+U 1 1 579CC622
+P 10600 1550
+F 0 "P?" H 10600 1700 50  0000 C CNN
+F 1 "CONN_01X02" V 10700 1550 50  0000 C CNN
+F 2 "" H 10600 1550 60  0000 C CNN
+F 3 "" H 10600 1550 60  0000 C CNN
+	1    10600 1550
+	1    0    0    -1
+$EndComp
+$Comp
+L GND #PWR?
+U 1 1 579CC6F3
+P 10200 1750
+F 0 "#PWR?" H 10200 1500 50  0001 C CNN
+F 1 "GND" H 10200 1600 50  0000 C CNN
+F 2 "" H 10200 1750 60  0000 C CNN
+F 3 "" H 10200 1750 60  0000 C CNN
+	1    10200 1750
+	1    0    0    -1
+$EndComp
+Wire Wire Line
+	10200 1750 10200 1600
+Wire Wire Line
+	10200 1600 10400 1600
+Wire Wire Line
+	10400 1500 9650 1500
+Text Label 9800 1500 0    60   ~ 0
+~EXT_TRIGGER
+$Comp
+L SD103A D?
+U 1 1 579CC905
+P 9650 1350
+F 0 "D?" H 9650 1450 50  0000 C CNN
+F 1 "SD103A" H 9650 1250 50  0000 C CNN
+F 2 "" H 9650 1350 60  0000 C CNN
+F 3 "" H 9650 1350 60  0000 C CNN
+	1    9650 1350
+	0    1    1    0
+$EndComp
+$Comp
+L SD103A D?
+U 1 1 579CC9BB
+P 9650 1650
+F 0 "D?" H 9650 1750 50  0000 C CNN
+F 1 "SD103A" H 9650 1550 50  0000 C CNN
+F 2 "" H 9650 1650 60  0000 C CNN
+F 3 "" H 9650 1650 60  0000 C CNN
+	1    9650 1650
+	0    1    1    0
+$EndComp
+$Comp
+L GND #PWR?
+U 1 1 579CCA37
+P 9650 1800
+F 0 "#PWR?" H 9650 1550 50  0001 C CNN
+F 1 "GND" H 9650 1650 50  0000 C CNN
+F 2 "" H 9650 1800 60  0000 C CNN
+F 3 "" H 9650 1800 60  0000 C CNN
+	1    9650 1800
+	1    0    0    -1
+$EndComp
+$Comp
+L +3.3V #PWR?
+U 1 1 579CCA9B
+P 9650 1200
+F 0 "#PWR?" H 9650 1050 50  0001 C CNN
+F 1 "+3.3V" H 9650 1340 50  0000 C CNN
+F 2 "" H 9650 1200 60  0000 C CNN
+F 3 "" H 9650 1200 60  0000 C CNN
+	1    9650 1200
+	1    0    0    -1
+$EndComp
+Connection ~ 9650 1500
 $EndSCHEMATC
